Commit message: Refactor code structure for improved readability and maintainability

File: config/dual_fr3.gazebo.urdf.xacro (robot description, xacro)
@@ -3,22 +3,26 @@
   <xacro:include filename="$(find franka_description)/robots/common/franka_robot.xacro"/>
   <xacro:include filename="$(find franka_hardware)/ros2_control/franka_arm.ros2_control.xacro"/>
+  <xacro:include filename="$(find dual_fr3_moveit_config)/config/research_franka_hand.xacro"/>
   <xacro:arg name="load_gripper" default="true"/>
   <xacro:arg name="ee_id" default="franka_hand"/>
   <xacro:arg name="arm_yaw" default="0"/>
   <xacro:arg name="gazebo_effort" default="true"/>
-  <material name="worktable_dark_green">
-    <color rgba="0.0 0.22 0.15 1.0"/>
+  <material name="fixture_blue_gray">
+    <color rgba="0.7921568627 0.8196078431 0.9333333333 1.0"/>
+  </material>
+  <material name="fixture_white">
+    <color rgba="1.0 1.0 1.0 1.0"/>
   </material>
   <link name="world"/>
   <link name="worktable">
     <visual>
-      <origin xyz="0.375 0.75 -0.025" rpy="0 0 0"/>
+      <origin xyz="0.375 0.75 -0.02" rpy="0 0 0"/>
       <geometry>
-        <box size="0.75 1.5 0.05"/>
+        <mesh filename="package://dual_fr3_moveit_config/meshes/base_link.STL"/>
       </geometry>
-      <material name="worktable_dark_green"/>
+      <material name="fixture_blue_gray"/>
     </visual>
     <collision>
-      <origin xyz="0.375 0.75 -0.030" rpy="0 0 0"/>
+      <origin xyz="0.375 0.75 -0.02" rpy="0 0 0"/>
       <geometry>
         <box size="0.75 1.5 0.04"/>
@@ -31,8 +35,58 @@
     </inertial>
   </link>
+  <link name="plate">
+    <visual>
+      <origin xyz="0 0 0" rpy="0 0 0"/>
+      <geometry>
+        <mesh filename="package://dual_fr3_moveit_config/meshes/Plate.STL"/>
+      </geometry>
+      <material name="fixture_blue_gray"/>
+    </visual>
+    <collision>
+      <origin xyz="0 0 0.025" rpy="0 0 0"/>
+      <geometry>
+        <box size="0.6 1.06 0.05"/>
+      </geometry>
+    </collision>
+    <inertial>
+      <origin xyz="0.0088197177 0.0000715269 0.0106850997" rpy="0 0 0"/>
+      <mass value="11.3852045210"/>
+      <inertia ixx="0.9160469835" ixy="0.0000187920" ixz="0.0" iyy="0.3327549084" iyz="0.0" izz="1.2478608782"/>
+    </inertial>
+  </link>
+  <link name="trunking">
+    <visual>
+      <origin xyz="0 0 0" rpy="0 0 0"/>
+      <geometry>
+        <mesh filename="package://dual_fr3_moveit_config/meshes/Trunking.STL"/>
+      </geometry>
+      <material name="fixture_white"/>
+    </visual>
+    <collision>
+      <origin xyz="0 0 0" rpy="0 0 0"/>
+      <geometry>
+        <mesh filename="package://dual_fr3_moveit_config/meshes/collision/trunking.STL"/>
+      </geometry>
+    </collision>
+    <inertial>
+      <origin xyz="-0.2685275817 -0.4514864586 0.0188180688" rpy="0 0 0"/>
+      <mass value="1.0228350951"/>
+      <inertia ixx="0.0268769452" ixy="-0.0000088301" ixz="-0.0000047833" iyy="0.0071799691" iyz="-0.0000585560" izz="0.0332373299"/>
+    </inertial>
+  </link>
   <joint name="world_to_worktable" type="fixed">
     <parent link="world"/>
     <child link="worktable"/>
     <origin xyz="0 0 0" rpy="0 0 0"/>
+  </joint>
+  <joint name="worktable_to_plate" type="fixed">
+    <parent link="worktable"/>
+    <child link="plate"/>
+    <origin xyz="0.5468955964 0.6484339463 -0.02" rpy="0 0 0"/>
+  </joint>
+  <joint name="plate_to_trunking" type="fixed">
+    <parent link="plate"/>
+    <child link="trunking"/>
+    <origin xyz="0.2621044036 0.4745660537 0.02" rpy="0 0 0"/>
   </joint>
   <joint name="worktable_to_left_fr3_mount" type="fixed">
@@ -49,5 +103,5 @@
       robot_type="fr3"
       parent="world"
-      hand="$(arg load_gripper)"
+      hand="false"
       ee_id="$(arg ee_id)"
       rpy_ee="0 0 ${-pi/4}"
@@ -64,5 +118,5 @@
       robot_type="fr3"
       parent="world"
-      hand="$(arg load_gripper)"
+      hand="false"
       ee_id="$(arg ee_id)"
       rpy_ee="0 0 ${-pi/4}"
@@ -76,4 +130,20 @@
       rpy="0 0 $(arg arm_yaw)"
       gazebo="true"/>
+  <xacro:if value="$(arg load_gripper)">
+    <xacro:research_franka_hand
+        connected_to="left_fr3_link8"
+        prefix="left_fr3_"
+        ee_inertials="${xacro.load_yaml('$(find franka_description)/end_effectors/franka_hand/inertials.yaml')}"
+        rpy_ee="0 0 ${-pi/4}"
+        tcp_xyz="0 0 0.1034"
+        tcp_rpy="0 0 0"/>
+    <xacro:research_franka_hand
+        connected_to="right_fr3_link8"
+        prefix="right_fr3_"
+        ee_inertials="${xacro.load_yaml('$(find franka_description)/end_effectors/franka_hand/inertials.yaml')}"
+        rpy_ee="0 0 ${-pi/4}"
+        tcp_xyz="0 0 0.1034"
+        tcp_rpy="0 0 0"/>
+  </xacro:if>
   <xacro:franka_arm_ros2_control
       robot_type="fr3"

File: config/dual_fr3.srdf.xacro (robot description, xacro)
@@ -98,3 +98,6 @@
   <disable_collisions link1="worktable" link2="left_fr3_link0" reason="Mount"/>
   <disable_collisions link1="worktable" link2="right_fr3_link0" reason="Mount"/>
+  <disable_collisions link1="worktable" link2="plate" reason="Adjacent"/>
+  <disable_collisions link1="worktable" link2="trunking" reason="Fixture"/>
+  <disable_collisions link1="plate" link2="trunking" reason="Adjacent"/>
 </robot>

File: config/dual_fr3.urdf.xacro (robot description, xacro)
@@ -3,4 +3,5 @@
   <xacro:include filename="$(find franka_description)/robots/common/franka_robot.xacro"/>
   <xacro:include filename="$(find franka_hardware)/ros2_control/franka_arm.ros2_control.xacro"/>
+  <xacro:include filename="$(find dual_fr3_moveit_config)/config/research_franka_hand.xacro"/>
   <xacro:arg name="use_fake_hardware" default="true"/>
   <xacro:arg name="fake_sensor_commands" default="false"/>
@@ -10,21 +11,53 @@
   <xacro:arg name="ee_id" default="franka_hand"/>
   <xacro:arg name="arm_yaw" default="0"/>
-  <material name="worktable_dark_green">
-    <color rgba="0.0 0.22 0.15 1.0"/>
+  <material name="fixture_blue_gray">
+    <color rgba="0.7921568627 0.8196078431 0.9333333333 1.0"/>
+  </material>
+  <material name="fixture_white">
+    <color rgba="1.0 1.0 1.0 1.0"/>
   </material>
   <link name="world"/>
   <link name="worktable">
     <visual>
-      <origin xyz="0.375 0.75 -0.025" rpy="0 0 0"/>
+      <origin xyz="0.375 0.75 -0.02" rpy="0 0 0"/>
       <geometry>
-        <box size="0.75 1.5 0.05"/>
+        <mesh filename="package://dual_fr3_moveit_config/meshes/base_link.STL"/>
       </geometry>
-      <material name="worktable_dark_green"/>
+      <material name="fixture_blue_gray"/>
     </visual>
-    <!-- Keep the collision top slightly below the visual top to avoid startup contact at the mounts. -->
     <collision>
-      <origin xyz="0.375 0.75 -0.030" rpy="0 0 0"/>
+      <origin xyz="0.375 0.75 -0.02" rpy="0 0 0"/>
       <geometry>
         <box size="0.75 1.5 0.04"/>
+      </geometry>
+    </collision>
+  </link>
+  <link name="plate">
+    <visual>
+      <origin xyz="0 0 0" rpy="0 0 0"/>
+      <geometry>
+        <mesh filename="package://dual_fr3_moveit_config/meshes/Plate.STL"/>
+      </geometry>
+      <material name="fixture_blue_gray"/>
+    </visual>
+    <collision>
+      <origin xyz="0 0 0.025" rpy="0 0 0"/>
+      <geometry>
+        <box size="0.6 1.06 0.05"/>
+      </geometry>
+    </collision>
+  </link>
+  <link name="trunking">
+    <visual>
+      <origin xyz="0 0 0" rpy="0 0 0"/>
+      <geometry>
+        <mesh filename="package://dual_fr3_moveit_config/meshes/Trunking.STL"/>
+      </geometry>
+      <material name="fixture_white"/>
+    </visual>
+    <collision>
+      <origin xyz="0 0 0" rpy="0 0 0"/>
+      <geometry>
+        <mesh filename="package://dual_fr3_moveit_config/meshes/collision/trunking.STL"/>
       </geometry>
     </collision>
@@ -34,4 +67,14 @@
     <child link="worktable"/>
     <origin xyz="0 0 0" rpy="0 0 0"/>
+  </joint>
+  <joint name="worktable_to_plate" type="fixed">
+    <parent link="worktable"/>
+    <child link="plate"/>
+    <origin xyz="0.5468955964 0.6484339463 -0.02" rpy="0 0 0"/>
+  </joint>
+  <joint name="plate_to_trunking" type="fixed">
+    <parent link="plate"/>
+    <child link="trunking"/>
+    <origin xyz="0.2621044036 0.4745660537 0.02" rpy="0 0 0"/>
   </joint>
   <joint name="worktable_to_left_fr3_mount" type="fixed">
@@ -48,5 +91,5 @@
       robot_type="fr3"
       parent="world"
-      hand="$(arg load_gripper)"
+      hand="false"
       ee_id="$(arg ee_id)"
       rpy_ee="0 0 ${-pi/4}"
@@ -62,5 +105,5 @@
       robot_type="fr3"
       parent="world"
-      hand="$(arg load_gripper)"
+      hand="false"
       ee_id="$(arg ee_id)"
       rpy_ee="0 0 ${-pi/4}"
@@ -73,4 +116,20 @@
       connected_to="right_fr3_mount"
       rpy="0 0 $(arg arm_yaw)"/>
+  <xacro:if value="$(arg load_gripper)">
+    <xacro:research_franka_hand
+        connected_to="left_fr3_link8"
+        prefix="left_fr3_"
+        ee_inertials="${xacro.load_yaml('$(find franka_description)/end_effectors/franka_hand/inertials.yaml')}"
+        rpy_ee="0 0 ${-pi/4}"
+        tcp_xyz="0 0 0.1034"
+        tcp_rpy="0 0 0"/>
+    <xacro:research_franka_hand
+        connected_to="right_fr3_link8"
+        prefix="right_fr3_"
+        ee_inertials="${xacro.load_yaml('$(find franka_description)/end_effectors/franka_hand/inertials.yaml')}"
+        rpy_ee="0 0 ${-pi/4}"
+        tcp_xyz="0 0 0.1034"
+        tcp_rpy="0 0 0"/>
+  </xacro:if>
   <xacro:franka_arm_ros2_control
       robot_type="fr3"

Commit message: fix gazebo

File: config/dual_fr3.gazebo.urdf.xacro (robot description, xacro)
@@ -2,5 +2,4 @@
 <robot xmlns:xacro="http://www.ros.org/wiki/xacro" name="dual_fr3">
   <xacro:include filename="$(find franka_description)/robots/common/franka_robot.xacro"/>
-  <xacro:include filename="$(find franka_hardware)/ros2_control/franka_arm.ros2_control.xacro"/>
   <xacro:include filename="$(find dual_fr3_moveit_config)/config/research_franka_hand.xacro"/>
   <xacro:arg name="load_gripper" default="true"/>
@@ -102,4 +101,9 @@
   <xacro:franka_robot
       robot_type="fr3"
+      joint_limits="${xacro.load_yaml('$(find franka_description)/robots/fr3/joint_limits.yaml')}"
+      kinematics="${xacro.load_yaml('$(find franka_description)/robots/fr3/kinematics.yaml')}"
+      accelerometer_config="${xacro.load_yaml('$(find franka_description)/robots/fr3/accelerometers.yaml')}"
+      inertials="${xacro.load_yaml('$(find franka_description)/robots/fr3/inertials.yaml')}"
+      dynamics="${xacro.load_yaml('$(find franka_description)/robots/fr3/dynamics.yaml')}"
       parent="world"
       hand="false"
@@ -113,8 +117,12 @@
       arm_prefix="left_"
       connected_to="left_fr3_mount"
-      rpy="0 0 $(arg arm_yaw)"
-      gazebo="true"/>
+      rpy="0 0 $(arg arm_yaw)"/>
   <xacro:franka_robot
       robot_type="fr3"
+      joint_limits="${xacro.load_yaml('$(find franka_description)/robots/fr3/joint_limits.yaml')}"
+      kinematics="${xacro.load_yaml('$(find franka_description)/robots/fr3/kinematics.yaml')}"
+      accelerometer_config="${xacro.load_yaml('$(find franka_description)/robots/fr3/accelerometers.yaml')}"
+      inertials="${xacro.load_yaml('$(find franka_description)/robots/fr3/inertials.yaml')}"
+      dynamics="${xacro.load_yaml('$(find franka_description)/robots/fr3/dynamics.yaml')}"
       parent="world"
       hand="false"
@@ -128,6 +136,5 @@
       arm_prefix="right_"
       connected_to="right_fr3_mount"
-      rpy="0 0 $(arg arm_yaw)"
-      gazebo="true"/>
+      rpy="0 0 $(arg arm_yaw)"/>
   <xacro:if value="$(arg load_gripper)">
     <xacro:research_franka_hand
@@ -146,32 +153,46 @@
         tcp_rpy="0 0 0"/>
   </xacro:if>
-  <xacro:franka_arm_ros2_control
-      robot_type="fr3"
-      include_effort_command="$(arg gazebo_effort)"
-      include_finger_joint="false"
-      arm_prefix="left_">
-    <hardware_plugin>
+  <!--
+    Keep Gazebo control resources local to this simulation-only description.
+    The real-hardware description uses two independent controller managers and
+    must not inherit the single-manager layout used here.
+  -->
+  <xacro:macro name="gazebo_control_joint" params="name initial_position">
+    <joint name="${name}">
+      <command_interface name="position"/>
       <xacro:if value="$(arg gazebo_effort)">
-        <plugin>franka_gazebo_hardware/FrankaGazeboHardwareInterface</plugin>
+        <command_interface name="effort"/>
       </xacro:if>
-      <xacro:unless value="$(arg gazebo_effort)">
-        <plugin>gz_ros2_control/GazeboSimSystem</plugin>
-      </xacro:unless>
-    </hardware_plugin>
-  </xacro:franka_arm_ros2_control>
-  <xacro:franka_arm_ros2_control
-      robot_type="fr3"
-      include_effort_command="$(arg gazebo_effort)"
-      include_finger_joint="false"
-      arm_prefix="right_">
-    <hardware_plugin>
-      <xacro:if value="$(arg gazebo_effort)">
-        <plugin>franka_gazebo_hardware/FrankaGazeboHardwareInterface</plugin>
-      </xacro:if>
-      <xacro:unless value="$(arg gazebo_effort)">
-        <plugin>gz_ros2_control/GazeboSimSystem</plugin>
-      </xacro:unless>
-    </hardware_plugin>
-  </xacro:franka_arm_ros2_control>
+      <state_interface name="position">
+        <param name="initial_value">${initial_position}</param>
+      </state_interface>
+      <state_interface name="velocity"/>
+      <state_interface name="effort"/>
+    </joint>
+  </xacro:macro>
+  <ros2_control name="dual_fr3_gazebo_system" type="system">
+    <hardware>
+      <plugin>gz_ros2_control/GazeboSimSystem</plugin>
+    </hardware>
+    <xacro:gazebo_control_joint name="left_fr3_joint1" initial_position="0.0"/>
+    <xacro:gazebo_control_joint name="left_fr3_joint2" initial_position="${-pi/4}"/>
+    <xacro:gazebo_control_joint name="left_fr3_joint3" initial_position="0.0"/>
+    <xacro:gazebo_control_joint name="left_fr3_joint4" initial_position="${-3*pi/4}"/>
+    <xacro:gazebo_control_joint name="left_fr3_joint5" initial_position="0.0"/>
+    <xacro:gazebo_control_joint name="left_fr3_joint6" initial_position="${pi/2}"/>
+    <xacro:gazebo_control_joint name="left_fr3_joint7" initial_position="${pi/4}"/>
+    <xacro:gazebo_control_joint name="right_fr3_joint1" initial_position="0.0"/>
+    <xacro:gazebo_control_joint name="right_fr3_joint2" initial_position="${-pi/4}"/>
+    <xacro:gazebo_control_joint name="right_fr3_joint3" initial_position="0.0"/>
+    <xacro:gazebo_control_joint name="right_fr3_joint4" initial_position="${-3*pi/4}"/>
+    <xacro:gazebo_control_joint name="right_fr3_joint5" initial_position="0.0"/>
+    <xacro:gazebo_control_joint name="right_fr3_joint6" initial_position="${pi/2}"/>
+    <xacro:gazebo_control_joint name="right_fr3_joint7" initial_position="${pi/4}"/>
+    <!-- The second finger joint follows joint1 through the URDF mimic tag. -->
+    <xacro:if value="$(arg load_gripper)">
+      <xacro:gazebo_control_joint name="left_fr3_finger_joint1" initial_position="0.04"/>
+      <xacro:gazebo_control_joint name="right_fr3_finger_joint1" initial_position="0.04"/>
+    </xacro:if>
+  </ros2_control>
   <gazebo>
     <plugin filename="gz_ros2_control-system" name="gz_ros2_control::GazeboSimROS2ControlPlugin">

Commit message: update tcp

File: config/dual_fr3.gazebo.urdf.xacro (robot description, xacro)
@@ -136,5 +136,5 @@
         ee_inertials="${xacro.load_yaml('$(find franka_description)/end_effectors/franka_hand/inertials.yaml')}"
         rpy_ee="0 0 ${-pi/4}"
-        tcp_xyz="0 0 0.1034"
+        tcp_xyz="0 0 0.1524"
         tcp_rpy="0 0 0"/>
     <xacro:research_franka_hand
@@ -143,5 +143,5 @@
         ee_inertials="${xacro.load_yaml('$(find franka_description)/end_effectors/franka_hand/inertials.yaml')}"
         rpy_ee="0 0 ${-pi/4}"
-        tcp_xyz="0 0 0.1034"
+        tcp_xyz="0 0 0.1524"
         tcp_rpy="0 0 0"/>
   </xacro:if>

File: config/dual_fr3.urdf.xacro (robot description, xacro)
@@ -122,5 +122,5 @@
         ee_inertials="${xacro.load_yaml('$(find franka_description)/end_effectors/franka_hand/inertials.yaml')}"
         rpy_ee="0 0 ${-pi/4}"
-        tcp_xyz="0 0 0.1034"
+        tcp_xyz="0 0 0.1524"
         tcp_rpy="0 0 0"/>
     <xacro:research_franka_hand
@@ -129,5 +129,5 @@
         ee_inertials="${xacro.load_yaml('$(find franka_description)/end_effectors/franka_hand/inertials.yaml')}"
         rpy_ee="0 0 ${-pi/4}"
-        tcp_xyz="0 0 0.1034"
+        tcp_xyz="0 0 0.1524"
         tcp_rpy="0 0 0"/>
   </xacro:if>

File: config/research_franka_hand.xacro (robot description, xacro)
@@ -6,5 +6,5 @@
                        rpy_ee:='0 0 0'
                        xyz_ee:='0 0 0'
-                       tcp_xyz:='0 0 0.1034'
+                       tcp_xyz:='0 0 0.1524'
                        tcp_rpy:='0 0 0'">
     <joint name="${prefix}hand_joint" type="fixed">
@@ -43,7 +43,7 @@
       </visual>
       <collision name="${prefix}leftfinger_collision">
-        <origin xyz="0 0.0135 0.05545" rpy="0 0 0"/>
+        <origin xyz="0 0 0.0964" rpy="0 0 0"/>
         <geometry>
-          <box size="0.021 0.029 0.106"/>
+          <mesh filename="package://dual_fr3_moveit_config/meshes/research_finger/finger.STL"/>
         </geometry>
       </collision>
@@ -61,7 +61,7 @@
       </visual>
       <collision name="${prefix}rightfinger_collision">
-        <origin xyz="0 0.0135 0.05545" rpy="0 0 0"/>
+        <origin xyz="0 0 0.0964" rpy="0 0 0"/>
         <geometry>
-          <box size="0.021 0.029 0.106"/>
+          <mesh filename="package://dual_fr3_moveit_config/meshes/research_finger/finger.STL"/>
         </geometry>
       </collision>

Commit message: update tcp

File: config/dual_fr3.gazebo.urdf.xacro (robot description, xacro)
@@ -143,5 +143,5 @@
         ee_inertials="${xacro.load_yaml('$(find franka_description)/end_effectors/franka_hand/inertials.yaml')}"
         rpy_ee="0 0 ${-pi/4}"
-        tcp_xyz="0 0 0.1034"
+        tcp_xyz="0 0 0.1524"
         tcp_rpy="0 0 0"/>
     <xacro:research_franka_hand
@@ -150,5 +150,5 @@
         ee_inertials="${xacro.load_yaml('$(find franka_description)/end_effectors/franka_hand/inertials.yaml')}"
         rpy_ee="0 0 ${-pi/4}"
-        tcp_xyz="0 0 0.1034"
+        tcp_xyz="0 0 0.1524"
         tcp_rpy="0 0 0"/>
   </xacro:if>

File: config/dual_fr3.urdf.xacro (robot description, xacro)
@@ -134,5 +134,5 @@
         ee_inertials="${xacro.load_yaml('$(find franka_description)/end_effectors/franka_hand/inertials.yaml')}"
         rpy_ee="0 0 ${-pi/4}"
-        tcp_xyz="0 0 0.1034"
+        tcp_xyz="0 0 0.1524"
         tcp_rpy="0 0 0"/>
     <xacro:research_franka_hand
@@ -141,5 +141,5 @@
         ee_inertials="${xacro.load_yaml('$(find franka_description)/end_effectors/franka_hand/inertials.yaml')}"
         rpy_ee="0 0 ${-pi/4}"
-        tcp_xyz="0 0 0.1034"
+        tcp_xyz="0 0 0.1524"
         tcp_rpy="0 0 0"/>
   </xacro:if>

File: config/research_franka_hand.xacro (robot description, xacro)
@@ -6,5 +6,5 @@
                        rpy_ee:='0 0 0'
                        xyz_ee:='0 0 0'
-                       tcp_xyz:='0 0 0.1034'
+                       tcp_xyz:='0 0 0.1524'
                        tcp_rpy:='0 0 0'">
     <joint name="${prefix}hand_joint" type="fixed">
@@ -43,7 +43,7 @@
       </visual>
       <collision name="${prefix}leftfinger_collision">
-        <origin xyz="0 0.0135 0.05545" rpy="0 0 0"/>
+        <origin xyz="0 0 0.0964" rpy="0 0 0"/>
         <geometry>
-          <box size="0.021 0.029 0.106"/>
+          <mesh filename="package://dual_fr3_moveit_config/meshes/research_finger/finger.STL"/>
         </geometry>
       </collision>
@@ -61,7 +61,7 @@
       </visual>
       <collision name="${prefix}rightfinger_collision">
-        <origin xyz="0 0.0135 0.05545" rpy="0 0 0"/>
+        <origin xyz="0 0 0.0964" rpy="0 0 0"/>
         <geometry>
-          <box size="0.021 0.029 0.106"/>
+          <mesh filename="package://dual_fr3_moveit_config/meshes/research_finger/finger.STL"/>
         </geometry>
       </collision>

Commit message: fix plan arguements

File: config/dual_fr3.gazebo.urdf.xacro (robot description, xacro)
@@ -65,5 +65,5 @@
       <origin xyz="0 0 0" rpy="0 0 0"/>
       <geometry>
-        <mesh filename="package://dual_fr3_moveit_config/meshes/collision/trunking.STL"/>
+        <mesh filename="package://dual_fr3_moveit_config/meshes/Trunking.STL"/>
       </geometry>
     </collision>

File: config/dual_fr3.urdf.xacro (robot description, xacro)
@@ -61,5 +61,5 @@
       <origin xyz="0 0 0" rpy="0 0 0"/>
       <geometry>
-        <mesh filename="package://dual_fr3_moveit_config/meshes/collision/trunking.STL"/>
+        <mesh filename="package://dual_fr3_moveit_config/meshes/Trunking.STL"/>
       </geometry>
     </collision>

Commit message: feat: integrate Rope-Actor cable simulation with ROS/MTC, stabilize mesh contacts and adaptive stepping

File: config/dual_fr3.gazebo.urdf.xacro (robot description, xacro)
@@ -54,16 +54,17 @@
     </inertial>
   </link>
+  <!-- Compensate the simplified CAD export origin; keep the existing fixture layout. -->
   <link name="trunking">
     <visual>
-      <origin xyz="0 0 0" rpy="0 0 0"/>
-      <geometry>
-        <mesh filename="package://dual_fr3_moveit_config/meshes/Trunking.STL"/>
+      <origin xyz="0.00014546 -0.00068397 0" rpy="0 0 0"/>
+      <geometry>
+        <mesh filename="package://dual_fr3_moveit_config/meshes/Trunking_simplify.stl"/>
       </geometry>
       <material name="fixture_white"/>
     </visual>
     <collision>
-      <origin xyz="0 0 0" rpy="0 0 0"/>
-      <geometry>
-        <mesh filename="package://dual_fr3_moveit_config/meshes/Trunking.STL"/>
+      <origin xyz="0.00014546 -0.00068397 0" rpy="0 0 0"/>
+      <geometry>
+        <mesh filename="package://dual_fr3_moveit_config/meshes/Trunking_simplify.stl"/>
       </geometry>
     </collision>

File: config/dual_fr3.urdf.xacro (robot description, xacro)
@@ -50,16 +50,17 @@
     </collision>
   </link>
+  <!-- Compensate the simplified CAD export origin; keep the existing fixture layout. -->
   <link name="trunking">
     <visual>
-      <origin xyz="0 0 0" rpy="0 0 0"/>
+      <origin xyz="0.00014546 -0.00068397 0" rpy="0 0 0"/>
       <geometry>
-        <mesh filename="package://dual_fr3_moveit_config/meshes/Trunking.STL"/>
+        <mesh filename="package://dual_fr3_moveit_config/meshes/Trunking_simplify.stl"/>
       </geometry>
       <material name="fixture_white"/>
     </visual>
     <collision>
-      <origin xyz="0 0 0" rpy="0 0 0"/>
+      <origin xyz="0.00014546 -0.00068397 0" rpy="0 0 0"/>
       <geometry>
-        <mesh filename="package://dual_fr3_moveit_config/meshes/Trunking.STL"/>
+        <mesh filename="package://dual_fr3_moveit_config/meshes/Trunking_simplify.stl"/>
       </geometry>
     </collision>
